File: DAS24-ESP32/untitled.sch (EAGLE design)
At the start: 248 parts, among them IC1 MCP23017SS, IC4 MCP23017SS, J1 10118193-0001LF, K1 SRD-05VDC-SL-C, Q1 S9013, Q2 12MHz, Q3 MMBT3904, Q4 MMBT3904, Q5 S9013, Q6 S9013, U1 CH340G, U2 AMS1117, U3 ESP32-WROOM-32D, U4 PC817X2NIP0F, U49 PC817X2NIP0F, U5 PC817X2NIP0F, X1 MSTBA12, X2 MSTBA12, X5 MSTBA3, X6 MSTBA3, X7 MSTBA2, X8 MSTBA2

Commit message: pengajuan das dan revisi 21/02/2023
Parts:
- added 2: 330, rcl:R-EU_R0805
- added 3: 10k, rcl:R-EU_R0805
- added D56: US1M-13, US1M-13:US1M-13
- added JP1: (no value), adafruit:PINHD-1X6CLEAN
- added K2: 351, relay:351
- added Q7: S9013, S9013:S9013
- added U6: PC817X2NIP0F, PC817X2NIP0F:PC817X2NIP0F
- 1: value (none) -> 330
Connections:
- new net COMM1: K22.P, OPTO1.C, OPTO10.C, OPTO11.C, OPTO12.C, OPTO13.C, OPTO14.C, OPTO15.C, OPTO16.C, OPTO17.C, OPTO18.C, OPTO19.C, OPTO2.C, OPTO20.C, OPTO21.C, OPTO22.C, OPTO23.C, OPTO24.C, OPTO3.C, OPTO4.C, OPTO5.C, OPTO6.C, OPTO7.C, OPTO8.C, OPTO9.C, Z1.A, Z10.A, Z11.A, Z12.A, Z13.A, Z14.A, Z15.A, Z16.A, Z17.A, Z18.A, Z19.A, Z2.A, Z20.A, Z21.A, Z22.A, Z23.A, Z24.A, Z3.A, Z4.A, Z5.A, Z6.A, Z7.A, Z8.A, Z9.A
- new net GND_TEST: 2.2, U3.IO27
- new net INT_LAN: U$1.INT, U3.IO32
- new net N$14: 2.1, U6.A
- new net N$18: 3.2, U6.CT
- new net N$23: D56.A, K21.2, Q7.C
- new net N$25: Q7.B, U6.ET
- net COMM: now also K22.O; no longer OPTO1.C, OPTO10.C, OPTO11.C, OPTO12.C, OPTO13.C, OPTO14.C, OPTO15.C, OPTO16.C, OPTO17.C, OPTO18.C, OPTO19.C, OPTO2.C, OPTO20.C, OPTO21.C, OPTO22.C, OPTO23.C, OPTO24.C, OPTO3.C, OPTO4.C, OPTO5.C, OPTO6.C, OPTO7.C, OPTO8.C, OPTO9.C, Z1.A, Z10.A, Z11.A, Z12.A, Z13.A, Z14.A, Z15.A, Z16.A, Z17.A, Z18.A, Z19.A, Z2.A, Z20.A, Z21.A, Z22.A, Z23.A, Z24.A, Z3.A, Z4.A, Z5.A, Z6.A, Z7.A, Z8.A, Z9.A
- net GND: now also JP1.1, K22.S, Q7.E, U6.C
- net OUT+: now also 3.1, D56.K, K21.1
- net SCL: now also JP1.4
- net SDA: now also JP1.3
- net VCC: now also JP1.2
